Commit message: URDF finished (hopefully), new Rviz settings

File: BCI/src/bci_sim_arm/urdf/bci_arm.urdf (robot description, URDF)
Before this commit: robot bci_arm, 16 links, 14 joints
Links:
- link index1: geometry visual cylinder length=2 radius=0.5
- link index2: geometry visual cylinder length=1 radius=0.5
- link index3: geometry visual cylinder length=1 radius=0.5
- link middle1: geometry visual cylinder length=2 radius=0.5
- link middle2: geometry visual cylinder length=1 radius=0.5
- link middle3: geometry visual cylinder length=1 radius=0.5
- link pinky1: geometry visual cylinder length=2 radius=0.5
- link pinky2: geometry visual cylinder length=1 radius=0.5
- link pinky3: geometry visual cylinder length=1 radius=0.5
- link ring1: geometry visual cylinder length=2 radius=0.5
- link ring2: geometry visual cylinder length=1 radius=0.5
- link ring3: geometry visual cylinder length=1 radius=0.5
- link thumb1: geometry visual box size=2 4 0.5
- link thumb2: geometry visual cylinder length=2 radius=1
- link thumb3: geometry visual cylinder length=1 radius=1
Joints:
- added joint second_middle_joint: type revolute, parent middle2, child middle3, origin xyz=0 2 0 rpy=0 0 0, axis 0 1 0, limit lower=0.0 upper=0.785 effort=100 velocity=0.5
- joint base_index_joint: axis 0 0 0 -> 3.75 6.5 0; limit (none) -> lower=0.0 upper=0.785 effort=100 velocity=0.5; origin xyz=2.25 2.75 0 rpy=0 0 0 -> xyz=3.75 8 0 rpy=0 0 0
- joint base_middle_joint: axis 0 0 0 -> 1.25 6.5 0; limit (none) -> lower=0.0 upper=0.785 effort=100 velocity=0.5; origin xyz=0.75 2.75 0 rpy=0 0 0 -> xyz=1.25 8 0 rpy=0 0 0
- joint base_pinky_joint: axis 0 0 0 -> -3.75 6 0; limit (none) -> lower=0.0 upper=0.785 effort=100 velocity=0.5; origin xyz=-2.25 2.75 0 rpy=0 0 0 -> xyz=-3.75 8 0 rpy=0 0 0
- joint base_ring_joint: axis 0 0 0 -> -1.25 6.5 0; limit (none) -> lower=0.0 upper=0.785 effort=100 velocity=0.5; origin xyz=-0.75 2.75 0 rpy=0 0 0 -> xyz=-1.25 8 0 rpy=0 0 0
- joint base_thumb_joint: axis 0 0 0 -> 6 0 0; limit (none) -> lower=0.0 upper=0.785 effort=100 velocity=0.5; origin xyz=3.5 0 0 rpy=0 0 0 -> xyz=8  0 0 rpy=0 0 0
- joint first_index_joint: axis 0 0 0 -> 0 1.5 0; limit (none) -> lower=0.0 upper=0.785 effort=100 velocity=0.5; origin xyz=0 1.25 0 rpy=0 0 0 -> xyz=0 2.5 0 rpy=0 0 0
- joint first_middle_joint: axis 0 0 0 -> 0 1.5 0; limit (none) -> lower=0.0 upper=0.785 effort=100 velocity=0.5; origin xyz=0 1.25 0 rpy=0 0 0 -> xyz=0 2.5 0 rpy=0 0 0
- joint first_pinky_joint: axis 0 0 0 -> 0 1.5 0; limit (none) -> lower=0.0 upper=0.785 effort=100 velocity=0.5; origin xyz=0 1.25 0 rpy=0 0 0 -> xyz=0 2.5 0 rpy=0 0 0
- joint first_ring_joint: axis 0 0 0 -> 0 1.5 0; limit (none) -> lower=0.0 upper=0.785 effort=100 velocity=0.5; origin xyz=0 1.25 0 rpy=0 0 0 -> xyz=0 2.5 0 rpy=0 0 0
- joint first_thumb_joint: axis 0 0 0 -> 0 2.5 0; limit (none) -> lower=0.0 upper=0.785 effort=100 velocity=0.5; origin xyz=0 2.25 0 rpy=0 0 0 -> xyz=0 4 0 rpy=0 0 0
- joint second_index_joint: axis 0 0 0 -> 0 1 0; limit (none) -> lower=0.0 upper=0.785 effort=100 velocity=0.5; origin xyz=0 0.75 0 rpy=0 0 0 -> xyz=0 2 0 rpy=0 0 0
- joint second_pinky_joint: axis 0 0 0 -> 0 1 0; limit (none) -> lower=0.0 upper=0.785 effort=100 velocity=0.5; origin xyz=0 0.75 0 rpy=0 0 0 -> xyz=0 2 0 rpy=0 0 0
- joint second_ring_joint: axis 0 0 0 -> 0 1 0; limit (none) -> lower=0.0 upper=0.785 effort=100 velocity=0.5; origin xyz=0 0.75 0 rpy=0 0 0 -> xyz=0 2 0 rpy=0 0 0
- joint second_thumb_joint: axis 0 0 0 -> 0 1.5 0; child middle3 -> thumb3; limit (none) -> lower=0.0 upper=0.785 effort=100 velocity=0.5; origin xyz=0 0.75 0 rpy=0 0 0 -> xyz=0 3 0 rpy=0 0 0; parent middle2 -> thumb2

Commit message: Arm finished (tested), fully articulated, GUI for rviz displayed, launch file finished

File: BCI/src/bci_sim_arm/urdf/bci_arm.urdf (robot description, URDF)
Before this commit: robot bci_arm, 16 links, 15 joints
Links:
- link base_link: geometry visual box size=10 12 2
- link thumb1: geometry visual box size=2 4 2
Joints:
- joint base_index_joint: axis 3.75 6.5 0 -> 1 0 0; origin xyz=3.75 8 0 rpy=0 0 0 -> xyz=3.75 8 0 rpy=1.57 0 0
- joint base_middle_joint: axis 1.25 6.5 0 -> 1 0 0; origin xyz=1.25 8 0 rpy=0 0 0 -> xyz=1.25 8 0 rpy=1.57 0 0
- joint base_pinky_joint: axis -3.75 6 0 -> 1 0 0; origin xyz=-3.75 8 0 rpy=0 0 0 -> xyz=-3.75 8 0 rpy=1.57 0 0
- joint base_ring_joint: axis -1.25 6.5 0 -> 1 0 0; origin xyz=-1.25 8 0 rpy=0 0 0 -> xyz=-1.25 8 0 rpy=1.57 0 0
- joint base_thumb_joint: axis 6 0 0 -> 0 1 0; limit lower=0.0 upper=0.785 effort=100 velocity=0.5 -> lower=-0.785 upper=0.0 effort=100 velocity=0.5; origin xyz=8  0 0 rpy=0 0 0 -> xyz=8 0 0 rpy=0 0 0
- joint first_index_joint: axis 0 1.5 0 -> 1 0 0; origin xyz=0 2.5 0 rpy=0 0 0 -> xyz=0 0 -2.5 rpy=0 0 0
- joint first_middle_joint: axis 0 1.5 0 -> 1 0 0; origin xyz=0 2.5 0 rpy=0 0 0 -> xyz=0 0 -2.5 rpy=0 0 0
- joint first_pinky_joint: axis 0 1.5 0 -> 1 0 0; origin xyz=0 2.5 0 rpy=0 0 0 -> xyz=0 0 -2.5 rpy=0 0 0
- joint first_ring_joint: axis 0 1.5 0 -> 1 0 0; origin xyz=0 2.5 0 rpy=0 0 0 -> xyz=0 0 -2.5 rpy=0 0 0
- joint first_thumb_joint: axis 0 2.5 0 -> 1 0 0; origin xyz=0 4 0 rpy=0 0 0 -> xyz=0 4 0 rpy=1.57 0 0
- joint second_index_joint: axis 0 1 0 -> 1 0 0; origin xyz=0 2 0 rpy=0 0 0 -> xyz=0 0 -2 rpy=0 0 0
- joint second_middle_joint: axis 0 1 0 -> 1 0 0; origin xyz=0 2 0 rpy=0 0 0 -> xyz=0 0 -2 rpy=0 0 0
- joint second_pinky_joint: axis 0 1 0 -> 1 0 0; origin xyz=0 2 0 rpy=0 0 0 -> xyz=0 0 -2 rpy=0 0 0
- joint second_ring_joint: axis 0 1 0 -> 1 0 0; origin xyz=0 2 0 rpy=0 0 0 -> xyz=0 0 -2 rpy=0 0 0
- joint second_thumb_joint: axis 0 1.5 0 -> 1 0 0; origin xyz=0 3 0 rpy=0 0 0 -> xyz=0 0 -3 rpy=0 0 0
